File: arduino_sequencer_schematic/_autosave-arduino_sequencer.sch (KiCad schematic (older format))
At the start: 174 parts, among them J1 AudioJack, J10 AudioJack, J11 AudioJack, J12 AudioJack, J13 AudioJack, J14 AudioJack, J15 AudioJack, J16 Conn_02x05, J2 AudioJack, J3 AudioJack, J4 AudioJack, J5 AudioJack, J6 AudioJack, J7 AudioJack, J8 AudioJack, J9 AudioJack, Q1 2N3904, Q10 2N3904, Q11 2N3904, Q2 2N3904, Q3 2N3904, Q4 2N3904, Q5 2N3904, Q6 2N3904, Q7 2N3904, Q8 2N3904, Q9 2N3904, SW1 SW_SPST, SW2 SW_Push, SW3 SW_Push, SW4 SW_Push, SW5 SW_SPST, SW6 SW_SPST, U1 74HC595, U2 TL084, U3 TL084, U4 L7805

Commit message: started PCB layout
Parts:
- removed J16: Conn_02x05, Connector_IDC:IDC-Header_2x05_P2.54mm_Vertical, symbol Connector_Generic:Conn_02x05_Counter_Clockwise
- added J16: Conn_02x05, Connector_IDC:IDC-Header_2x05_P2.54mm_Vertical, symbol Connector_Generic:Conn_02x05_Odd_Even
Connections:
- net GND: now also J16.4 (Pin_4), J16.6 (Pin_6), J16.8 (Pin_8)
- net at R64.1: now also J16.1 (Pin_1), J16.2 (Pin_2)
- net at C11.2, C7.1: now also J16.3 (Pin_3), J16.5 (Pin_5), J16.7 (Pin_7)
- net at R66.1: now also J16.10 (Pin_10), J16.9 (Pin_9)
Changed lines of the file:
@@
 Text GLabel 8400 2000 3    50   Output ~ 0
 INC_LED
-$Comp
-L Connector_Generic:Conn_02x05_Counter_Clockwise J16
-U 1 1 5FDF3CD0
-P 10050 10050
-F 0 "J16" H 10100 10500 50  0000 C CNN
-F 1 "Conn_02x05" H 10100 10400 50  0000 C CNN
-F 2 "Connector_IDC:IDC-Header_2x05_P2.54mm_Vertical" H 10050 10050 50  0001 C CNN
-F 3 "~" H 10050 10050 50  0001 C CNN
-	1    10050 10050
-	1    0    0    -1
-$EndComp
 Wire Wire Line
 	9850 9950 9850 10050
@@
 Wire Wire Line
 	2000 9550 2150 9550
+$Comp
+L Connector_Generic:Conn_02x05_Odd_Even J16
+U 1 1 604B4B47
+P 10050 10050
+F 0 "J16" H 10100 10500 50  0000 C CNN
+F 1 "Conn_02x05" H 10100 10400 50  0000 C CNN
+F 2 "Connector_IDC:IDC-Header_2x05_P2.54mm_Vertical" H 10050 10050 50  0001 C CNN
+F 3 "~" H 10050 10050 50  0001 C CNN
+	1    10050 10050
+	1    0    0    -1
+$EndComp
 $EndSCHEMATC
