File: arduino_sequencer_schematic/arduino_sequencer.kicad_pcb (KiCad board)
At the start: 2 copper layers, 174 parts, among them J1 AudioJack, J10 AudioJack, J11 AudioJack, J12 AudioJack, J13 AudioJack, J14 AudioJack, J15 AudioJack, J16 Conn_02x05, J2 AudioJack, J3 AudioJack, J4 AudioJack, J5 AudioJack, J6 AudioJack, J7 AudioJack, J8 AudioJack, J9 AudioJack, Q1 2N3904, Q10 2N3904, Q11 2N3904, Q2 2N3904, Q3 2N3904, Q4 2N3904, Q5 2N3904, Q6 2N3904, Q7 2N3904, Q8 2N3904, Q9 2N3904, SW1 SW_SPST, SW2 SW_Push, SW3 SW_Push, SW4 SW_Push, SW5 SW_SPST, SW6 SW_SPST, U1 74HC595, U2 TL084, U3 TL084, U4 L7805

Commit message: Changed gate voltage to 9V by default
Parts:
- added C3: 330nF, Capacitor_THT:CP_Radial_D10.0mm_P3.80mm, F.Cu at (88.0, 176.0)
- added C4: 100nF, Capacitor_THT:C_Disc_D6.0mm_W2.5mm_P5.00mm, F.Cu at (85.5, 161.5)
- added U1: L78L09_TO92, Package_TO_SOT_THT:TO-92_Inline, F.Cu at (98.0, 168.0)
- renumbered C8 to C10, C9 to C11, C10 to C12, C11 to C13, C3 to C5, C4 to C6, C5 to C7, C6 to C8, C7 to C9, R64 to R63, R63 to R64, U1 to U2, U2 to U3, U3 to U4, U4 to U5
Connections:
- A1 pad 27: V_GATE -> +5V
- C12 pad 2: V_GATE -> +5V
- D1 pad 2: V_GATE -> +5V
- R1 pad 2: V_GATE -> +5V
- R14 pad 2: V_GATE -> +5V
- R15 pad 1: V_GATE -> +5V
- R2 pad 1: V_GATE -> +5V
- R7 pad 2: V_GATE -> +5V
- R9 pad 1: V_GATE -> +5V
- U2 pad 10: V_GATE -> +5V
- U2 pad 16: V_GATE -> +5V
- U5 pad 3: V_GATE -> +5V
Routing:
- added copper zone on B.Cu, net +5V
- removed copper zone on B.Cu, net V_GATE

Commit message: Update arduino_sequencer.kicad_pcb
PCB updates
Parts:
- D1, D2, D26, D27, D28, D29, D30, D31, D32, D33, D34, D35, D36, D37, D4, D5, D6, D8, RV1, RV10, RV11, RV12, RV13, RV14, RV15, RV16, RV17, RV18, RV19, RV2, RV20, RV21, RV22, RV3, RV4, RV5, RV6, RV7, RV8, RV9, SW1, SW2, SW3, SW4, SW5, SW6: moved to B.Cu
- moved D10 544.5 mm to (-240.8, -45.2)
- moved D11 544.5 mm to (-224.2, -44.2)
- moved D12 544.5 mm to (-208.2, -45.8)
- moved D13 544.5 mm to (-191.8, -44.2)
- moved D14 544.5 mm to (-174.2, -44.8)
- moved D15 544.5 mm to (-159.2, -43.8)
- moved D16 544.5 mm to (-142.2, -44.8)
- moved D17 544.5 mm to (-124.8, -45.2)
- moved D18 544.5 mm to (-241.8, -18.8)
- moved D19 544.5 mm to (-225.8, -18.2)
- moved D20 544.5 mm to (-208.8, -17.8)
- moved D21 544.5 mm to (-191.8, -18.2)
- moved D22 544.5 mm to (-175.2, -18.8)
- moved D23 544.5 mm to (-158.8, -18.8)
- moved D24 544.5 mm to (-142.2, -18.2)
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Other:
- board outline added: 296 x 178 mm

Commit message: Update arduino_sequencer.kicad_pcb
PCB updates
Parts:
- moved C7 29.0 mm to (106.0, 215.0)
- moved C10 28.2 mm to (107.0, 85.2)
- moved C2 10.1 mm to (277.5, 108.0)
- moved C3 8.00 mm to (102.8, 143.5)
- moved C4 8.00 mm to (104.2, 156.5)
- moved U1 8.00 mm to (100.8, 156.5)
- moved D9 5.00 mm to (301.0, 219.5)
- moved R16 5.00 mm to (275.8, 219.5)
- moved R17 5.00 mm to (305.8, 219.5)
- moved C11 3.16 mm to (304.5, 148.2)
- moved C12 3.16 mm to (327.2, 150.5)
- moved U5 3.16 mm to (316.5, 151.2)
- moved Q3 1.41 mm to (291.0, 235.0)
- moved R18 1.41 mm to (296.0, 228.0)
- moved R65 0.75 mm to (114.0, 197.8)
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Other:
- outline, holes or cut-outs redrawn

Commit message: Update arduino_sequencer.kicad_pcb
pcb updates
Parts:
- moved RV6 502.7 mm to (251.9, 225.0), turned to 90 degrees
- moved RV7 490.8 mm to (286.0, 174.1), turned to 90 degrees
- moved D15 488.0 mm to (245.2, 229.2)
- moved RV1 487.6 mm to (223.1, 80.0), turned to 90 degrees
- moved RV14 481.0 mm to (261.6, 194.6), turned to 90 degrees
- moved R50 477.7 mm to (230.0, 88.5), turned to 270 degrees
- moved R34 477.2 mm to (225.0, 98.7), turned to 90 degrees
- moved D16 477.0 mm to (279.2, 178.5)
- moved RV5 474.9 mm to (191.9, 237.0), turned to 90 degrees
- moved RV13 473.9 mm to (220.2, 222.2), turned to 90 degrees
- moved R42 471.2 mm to (220.0, 98.7), turned to 90 degrees
- moved D10 470.9 mm to (217.0, 65.2)
- moved J6 468.7 mm to (223.5, 104.2), turned to 337.5 degrees
- moved R25 468.2 mm to (215.0, 88.5), turned to 270 degrees
- moved D22 460.0 mm to (213.8, 226.8)
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Other:
- outline, holes or cut-outs redrawn

Commit message: Update arduino_sequencer.kicad_pcb
pcb updates
Parts:
- moved R29 331.8 mm to (199.0, 216.2), turned to 90 degrees
- moved R30 323.1 mm to (249.0, 206.0), turned to 90 degrees
- moved Q8 321.5 mm to (206.0, 216.0), turned to 90 degrees
- moved Q9 313.4 mm to (256.0, 206.0), turned to 90 degrees
- moved R28 312.6 mm to (149.0, 195.0)
- moved Q7 309.9 mm to (150.0, 202.0)
- moved R38 301.8 mm to (188.8, 206.1), turned to 270 degrees
- moved R39 292.1 mm to (239.0, 195.8), turned to 270 degrees
- moved R37 282.7 mm to (159.2, 185.0), turned to 180 degrees
- moved R31 277.6 mm to (272.0, 159.0), turned to 180 degrees
- moved U2 271.8 mm to (243.0, 76.0)
- moved R40 265.9 mm to (261.8, 169.0)
- moved R27 260.6 mm to (139.0, 143.0)
- moved Q10 260.2 mm to (272.0, 152.0), turned to 180 degrees
- moved Q6 256.9 mm to (139.0, 150.0)
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Other:
- board text added: "1"
- board text added: "2"
- board text added: "3"
- board text added: "4"
- board text added: "5"
- board text added: "6"
- board text added: "7"
- board text added: "8"

Commit message: PCB routed
Parts:
- added J17: Conn_01x03, Connector_JST:JST_EH_B3B-EH-A_1x03_P2.50mm_Vertical, F.Cu at (274.0, 66.0)
- added REF**: PinHeader_1x15_P2.54mm_Vertical, Connector_PinHeader_2.54mm:PinHeader_1x15_P2.54mm_Vertical, F.Cu at (297.0, 126.0)
- added REF**: PinHeader_1x15_P2.54mm_Vertical, Connector_PinHeader_2.54mm:PinHeader_1x15_P2.54mm_Vertical, F.Cu at (297.0, 149.0)
- moved R6 23.7 mm to (317.7, 79.0), turned to 180 degrees
- moved R13 23.2 mm to (317.7, 105.8), turned to 180 degrees
- moved R12 22.6 mm to (307.5, 112.5)
- moved R5 20.7 mm to (307.5, 85.7)
- moved R7 19.7 mm to (317.7, 92.3)
- moved R18 19.7 mm to (315.7, 228.8), turned to 180 degrees
- moved Q3 16.8 mm to (296.0, 219.0), turned to 270 degrees
- moved R1 15.7 mm to (317.7, 65.5)
- moved R9 13.9 mm to (280.2, 108.8), turned to 0 degrees
- moved C2 13.6 mm to (287.8, 100.5), turned to 180 degrees
- moved C1 11.9 mm to (287.8, 74.5), turned to 180 degrees
- moved D3 11.7 mm to (307.5, 72.3), turned to 0 degrees
- moved J1 10.3 mm to (325.0, 80.0)
- moved J2 10.3 mm to (325.0, 110.0)
- moved R33 10.2 mm to (93.5, 68.0), turned to 0 degrees
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Connections:
- C13 pad 2: Net-(C13-Pad2) -> GND
- C9 pad 1: Net-(C13-Pad2) -> GND
- J16 pad 3: Net-(C13-Pad2) -> GND
- J16 pad 5: Net-(C13-Pad2) -> GND
- J16 pad 7: Net-(C13-Pad2) -> GND
Routing:
- net CV_OUT1: track 0.00 -> 515.3 mm
- net CV_OUT2: track 0.00 -> 493.5 mm
- net V_GATE: track 0.00 -> 463.7 mm
- net Net-(R28-Pad1): track 0.00 -> 365.7 mm, vias 0 -> 1
- net +12V: track 0.00 -> 294.1 mm
- net Net-(R29-Pad1): track 0.00 -> 281.8 mm, vias 0 -> 1
- net -12V: track 0.00 -> 234.5 mm
- net Net-(R27-Pad1): track 0.00 -> 222.7 mm, vias 0 -> 1
- net Net-(R30-Pad1): track 0.00 -> 201.6 mm, vias 0 -> 1
- net EXPANSION_LATCH: track 0.00 -> 161.2 mm
- net EXPANSION_CLOCK: track 0.00 -> 160.8 mm
- net FLIP_IN: track 0.00 -> 155.8 mm
- net Net-(R26-Pad1): track 0.00 -> 154.8 mm
- net CLOCK_IN: track 0.00 -> 149.3 mm
- net SER_DATA: track 0.00 -> 147.6 mm
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Other:
- board text added: "(Don´t sniff the magic smoke)"
- board text added: "30-12-2020"
- board text added: "Arduino Nano"
- board text added: "Arduino Sequencer"
- board text added: "DATA LATCH CLOCK"
- board text added: "JLCJLCJLCJLC"
- board text added: "PCB by TimMJN"

Commit message: Update arduino_sequencer.kicad_pcb
Other:
- board text added: "github.com/TimMJN"

Commit message: Footprint updates
Parts:
- removed REF** (x2): PinHeader_1x15_P2.54mm_Vertical, Connector_PinHeader_2.54mm:PinHeader_1x15_P2.54mm_Vertical
- A1: footprint Module:Arduino_Nano -> TimMJN:Arduino_Nano_2x_header
- SW2, SW3, SW4: footprint TimMJN:Mom_push_button -> TimMJN:Mom_push_button_PBS-110
Routing:
- net GND: track 112.3 -> 104.5 mm
- net +5V: track 27.9 -> 23.9 mm
- net Net-(A1-Pad30): track 4.01 -> 2.54 mm
- net Net-(A1-Pad28): track 4.01 -> 2.54 mm
- net Net-(A1-Pad26): track 4.01 -> 2.54 mm
- net Net-(A1-Pad25): track 4.01 -> 2.54 mm
- net Net-(A1-Pad24): track 4.01 -> 2.54 mm
- net Net-(A1-Pad23): track 4.01 -> 2.54 mm
- net Net-(A1-Pad22): track 4.01 -> 2.54 mm
- net Net-(A1-Pad21): track 4.01 -> 2.54 mm
- net Net-(A1-Pad20): track 4.01 -> 2.54 mm
- net Net-(A1-Pad19): track 4.01 -> 2.54 mm
- net Net-(A1-Pad18): track 4.01 -> 2.54 mm
- net Net-(A1-Pad17): track 4.01 -> 2.54 mm
- net Net-(A1-Pad16): track 4.01 -> 2.54 mm
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Other:
- board text removed: "Arduino Nano"
